Commit message: initial commit

File: urdf/robot.urdf (robot description, URDF)
Before this commit: robot summit_xl, 9 links, 8 joints
Links:
- removed link imu_link
- added link map
- added link odom
Joints:
- removed joint base_footprint_joint
- removed joint imu_joint
- added joint base_joint: type fixed, parent base_footprint, child base_link, origin xyz=0 0 0.010 rpy=0 0 0
- added joint map_to_odom: type fixed, parent map, child odom, origin xyz=0 0 0 rpy=0 0 0
- added joint odom_to_base_footprint: type fixed, parent odom, child base_footprint, origin xyz=0 0 0 rpy=0 0 0
- joint camera_joint: parent base_link -> lidar_link

Commit message: deleted files

File: urdf/robot.urdf (robot description, URDF)
Before this commit: robot summit_xl, 10 links, 9 joints
Links:
- removed link map
- removed link odom
- added link imu_link, mass 0.05; collision box size=0.05 0.05 0.02; visual box size=0.05 0.05 0.02
Joints:
- removed joint base_joint
- removed joint map_to_odom
- removed joint odom_to_base_footprint
- added joint base_footprint_joint: type fixed, parent base_link, child base_footprint, origin xyz=0 0 0 rpy=0 0 0
- added joint imu_joint: type fixed, parent base_link, child imu_link, origin xyz=0 0 0.05 rpy=0 0 0
- joint camera_joint: parent lidar_link -> base_link
